File: GuitarFX/_autosave-Codec.kicad_sch (KiCad schematic)
At the start: 79 parts, among them IC401 PCM3060PWR, J401 Screw_Terminal_01x04, U1 CS4272, U401 TLV9161IDBVR, U402 TLV9161IDBVR, U404 TLV9161IDBVR, U405 TLV9161IDBVR, U406 TLV9161IDBVR

Commit message: Fixed capactor value on frontend
Parts:
- added C437, C439: 1n, symbol Device:C
- added C438: 100n, symbol Device:C
- added C440: 150n, symbol Device:C
- added R434: 8.2k, symbol Device:R
- added R435: 27k, symbol Device:R
- added R436: 15k, symbol Device:R
- added U407: TLV9161IDBVR, SOT95P280X145-5N, symbol TLV9161IDBVR:TLV9161IDBVR
- C426: value 47u -> 22u
Connections:
- net +5VA: now also C436.1, C438.1, U407.5 (V+)
- net CODEC_VOUTL: now also R434.1
- net GND: now also C436.2, U402.2 (V-), U405.2 (V-), C438.2, C439.2, C440.2, U407.2 (V-)
- net IN_AA_BUFF_IN_L: now also C440.1, R436.2, U407.3 (+)
- net IN_AA_BUFF_OUT_L: now also C437.1, U407.1, U407.4 (-)
- new net: C439.1, R434.2, R435.1
- new net: C437.2, R435.2, R436.1
Other:
- note added: "3rd order Butterworth reconstruction filter. fc = 20kHz"
- note added: "Bias Generator"
- note added: "Rin = 500k (Parallel 1M resistors)"
- moved on the sheet: C411, C412, C413, C414, C415, C416, C417, C418, C419, C420, C421, C422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
