File: GuitarFX/Power.kicad_sch (KiCad schematic)
At the start: 20 parts, among them J201 Jack-DC, U3 NCP718xSN500, U4 NCP1117-3.3_SOT223

Commit message: Updated footprints for capacitors
Parts:
- C201, C202, C203, C204, C205, C206, C207, C208, C209, C210: footprint (none) -> Capacitor_SMD:C_0805_2012Metric
Changed lines of the file:
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@@
       (effects (font (size 1.27 1.27)) (justify left))
     )
-    (property "Footprint" "" (at 170.5102 73.025 0)
+    (property "Footprint" "Capacitor_SMD:C_0805_2012Metric" (at 170.5102 73.025 0)
       (effects (font (size 1.27 1.27)) hide)
     )
@@
       (effects (font (size 1.27 1.27)) (justify left))
     )
-    (property "Footprint" "" (at 192.1002 73.025 0)
+    (property "Footprint" "Capacitor_SMD:C_0805_2012Metric" (at 192.1002 73.025 0)
       (effects (font (size 1.27 1.27)) hide)
     )
@@
       (effects (font (size 1.27 1.27)) (justify left))
     )
-    (property "Footprint" "" (at 202.8952 73.025 0)
+    (property "Footprint" "Capacitor_SMD:C_0805_2012Metric" (at 202.8952 73.025 0)
       (effects (font (size 1.27 1.27)) hide)
     )
@@
       (effects (font (size 1.27 1.27)) (justify left))
     )
-    (property "Footprint" "" (at 118.4402 73.66 0)
+    (property "Footprint" "Capacitor_SMD:C_0805_2012Metric" (at 118.4402 73.66 0)
       (effects (font (size 1.27 1.27)) hide)
     )
@@
       (effects (font (size 1.27 1.27)) (justify left))
     )
-    (property "Footprint" "" (at 147.6502 113.03 0)
+    (property "Footprint" "Capacitor_SMD:C_0805_2012Metric" (at 147.6502 113.03 0)
       (effects (font (size 1.27 1.27)) hide)
     )
@@
       (effects (font (size 1.27 1.27)) (justify left))
     )
-    (property "Footprint" "" (at 119.0752 113.665 0)
+    (property "Footprint" "Capacitor_SMD:C_0805_2012Metric" (at 119.0752 113.665 0)
       (effects (font (size 1.27 1.27)) hide)
     )
@@
       (effects (font (size 1.27 1.27)) (justify left))
     )
-    (property "Footprint" "" (at 148.2852 73.66 0)
+    (property "Footprint" "Capacitor_SMD:C_0805_2012Metric" (at 148.2852 73.66 0)
       (effects (font (size 1.27 1.27)) hide)
     )
@@
       (effects (font (size 1.27 1.27)) (justify left))
     )
-    (property "Footprint" "" (at 103.2002 73.66 0)
+    (property "Footprint" "Capacitor_SMD:C_0805_2012Metric" (at 103.2002 73.66 0)
       (effects (font (size 1.27 1.27)) hide)
     )
@@
       (effects (font (size 1.27 1.27)) (justify left))
     )
-    (property "Footprint" "" (at 181.3052 73.025 0)
+    (property "Footprint" "Capacitor_SMD:C_0805_2012Metric" (at 181.3052 73.025 0)
       (effects (font (size 1.27 1.27)) hide)
     )
@@
       (effects (font (size 1.27 1.27)) (justify left))
     )
-    (property "Footprint" "" (at 88.5952 73.66 0)
-      (effects (font (size 1.27 1.27)) hide)
-    )
+    (property "Footprint" "Capacitor_SMD:C_0805_2012Metric" (at 88.5952 73.66 0)
+      (effects (font (size 1.27 1.27)) hide)
+    )
