File: GuitarFX/Codec.kicad_sch (KiCad schematic)
At the start: 85 parts, among them IC401 PCM3060PWR, J401 Screw_Terminal_01x04, U401 TLV9161IDBVR, U402 TLV9161IDBVR, U403 TLV9161IDBVR, U404 TLV9161IDBVR, U405 TLV9161IDBVR, U406 TLV9161IDBVR, U407 TLV9161IDBVR, U408 TLV9161IDBVR, U409 TLV9161IDBVR

Commit message: Changed butterworth filter components to 0603 for easier resoldering
Parts:
- C401, C408, C409, C410, C411, C416, C417, C418, C419, C424, C425, C435, C436: footprint Capacitor_SMD:C_0402_1005Metric -> Capacitor_SMD:C_0603_1608Metric
Changed lines of the file:
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@@
       (effects (font (size 1.27 1.27)))
     )
-    (property "Footprint" "Capacitor_SMD:C_0402_1005Metric" (at 139.3952 243.84 0)
+    (property "Footprint" "Capacitor_SMD:C_0603_1608Metric" (at 139.3952 243.84 0)
       (effects (font (size 1.27 1.27)) hide)
     )
@@
       (effects (font (size 1.27 1.27)))
     )
-    (property "Footprint" "Capacitor_SMD:C_0402_1005Metric" (at 180.6702 62.865 0)
+    (property "Footprint" "Capacitor_SMD:C_0603_1608Metric" (at 180.6702 62.865 0)
       (effects (font (size 1.27 1.27)) hide)
     )
@@
       (effects (font (size 1.27 1.27)))
     )
-    (property "Footprint" "Capacitor_SMD:C_0402_1005Metric" (at 139.3952 190.5 0)
+    (property "Footprint" "Capacitor_SMD:C_0603_1608Metric" (at 139.3952 190.5 0)
       (effects (font (size 1.27 1.27)) hide)
     )
@@
       (effects (font (size 1.27 1.27)))
     )
-    (property "Footprint" "Capacitor_SMD:C_0402_1005Metric" (at 80.9752 58.42 0)
+    (property "Footprint" "Capacitor_SMD:C_0603_1608Metric" (at 80.9752 58.42 0)
       (effects (font (size 1.27 1.27)) hide)
     )
@@
       (effects (font (size 1.27 1.27)))
     )
-    (property "Footprint" "Capacitor_SMD:C_0402_1005Metric" (at 144.145 159.0802 0)
+    (property "Footprint" "Capacitor_SMD:C_0603_1608Metric" (at 144.145 159.0802 0)
       (effects (font (size 1.27 1.27)) hide)
     )
@@
       (effects (font (size 1.27 1.27)))
     )
-    (property "Footprint" "Capacitor_SMD:C_0402_1005Metric" (at 154.6352 62.865 0)
+    (property "Footprint" "Capacitor_SMD:C_0603_1608Metric" (at 154.6352 62.865 0)
       (effects (font (size 1.27 1.27)) hide)
     )
@@
       (effects (font (size 1.27 1.27)))
     )
-    (property "Footprint" "Capacitor_SMD:C_0402_1005Metric" (at 113.3602 243.84 0)
+    (property "Footprint" "Capacitor_SMD:C_0603_1608Metric" (at 113.3602 243.84 0)
       (effects (font (size 1.27 1.27)) hide)
     )
@@
       (effects (font (size 1.27 1.27)))
     )
-    (property "Footprint" "Capacitor_SMD:C_0402_1005Metric" (at 185.42 87.3252 0)
+    (property "Footprint" "Capacitor_SMD:C_0603_1608Metric" (at 185.42 87.3252 0)
       (effects (font (size 1.27 1.27)) hide)
     )
@@
       (effects (font (size 1.27 1.27)))
     )
-    (property "Footprint" "Capacitor_SMD:C_0402_1005Metric" (at 180.6702 118.745 0)
+    (property "Footprint" "Capacitor_SMD:C_0603_1608Metric" (at 180.6702 118.745 0)
       (effects (font (size 1.27 1.27)) hide)
     )
@@
       (effects (font (size 1.27 1.27)))
     )
-    (property "Footprint" "Capacitor_SMD:C_0402_1005Metric" (at 185.42 31.4452 0)
+    (property "Footprint" "Capacitor_SMD:C_0603_1608Metric" (at 185.42 31.4452 0)
       (effects (font (size 1.27 1.27)) hide)
     )
@@
       (effects (font (size 1.27 1.27)))
     )
-    (property "Footprint" "Capacitor_SMD:C_0402_1005Metric" (at 154.6352 118.745 0)
+    (property "Footprint" "Capacitor_SMD:C_0603_1608Metric" (at 154.6352 118.745 0)
       (effects (font (size 1.27 1.27)) hide)
     )
@@
       (effects (font (size 1.27 1.27)))
     )
-    (property "Footprint" "Capacitor_SMD:C_0402_1005Metric" (at 80.9752 114.3 0)
+    (property "Footprint" "Capacitor_SMD:C_0603_1608Metric" (at 80.9752 114.3 0)
       (effects (font (size 1.27 1.27)) hide)
     )
@@
       (effects (font (size 1.27 1.27)))
     )
-    (property "Footprint" "Capacitor_SMD:C_0402_1005Metric" (at 144.145 212.4202 0)
+    (property "Footprint" "Capacitor_SMD:C_0603_1608Metric" (at 144.145 212.4202 0)
       (effects (font (size 1.27 1.27)) hide)
     )

Commit message: Changed to mono input, and finished rough Analog Frontend layout
Parts:
- removed C411, C417, C425, C435: 1n, Capacitor_SMD:C_0603_1608Metric, symbol Device:C
- removed C412, C413, C426, C427: 100n, Capacitor_SMD:C_0402_1005Metric, symbol Device:C
- removed C414: 10n, Capacitor_SMD:C_0402_1005Metric, symbol Device:C
- removed C415, C434: 4.7u, Capacitor_SMD:C_0603_1608Metric, symbol Device:C
- removed C416, C418, C436: 150p, Capacitor_SMD:C_0603_1608Metric, symbol Device:C
- removed D203 (x2): SMAJ15A, Diode_SMD:D_SMA, symbol Diode:SMAJ15A
- removed J401: Screw_Terminal_01x04, TerminalBlock_Phoenix:TerminalBlock_Phoenix_MPT-0,5-4-2.54_1x04_P2.54mm_Horizontal, symbol Connector:Screw_Terminal_01x04
- removed R411: 1k, Resistor_SMD:R_0402_1005Metric, symbol Device:R
- removed R412, R430: 8.2k, Resistor_SMD:R_0402_1005Metric, symbol Device:R
- removed R413, R431: 27k, Resistor_SMD:R_0402_1005Metric, symbol Device:R
- removed R414, R432: 15k, Resistor_SMD:R_0402_1005Metric, symbol Device:R
- removed R415, R433: 100R, Resistor_SMD:R_0402_1005Metric, symbol Device:R
- removed R416: 1M, Resistor_SMD:R_0402_1005Metric, symbol Device:R
- removed R434: 10k, Resistor_SMD:R_0402_1005Metric, symbol Device:R
- removed U404, U405, U408, U409: TLV9161IDBVR, TLV9161IDBVR:SOT95P280X145-5N, symbol TLV9161IDBVR:TLV9161IDBVR
- added J202 (x2): Screw_Terminal_01x02, TerminalBlock_Phoenix:TerminalBlock_Phoenix_MPT-0,5-2-2.54_1x02_P2.54mm_Horizontal, symbol Connector:Screw_Terminal_01x02
- C401, C419: footprint Capacitor_SMD:C_0603_1608Metric -> Capacitor_SMD:C_0402_1005Metric
- R405, R406, R407, R421, R422, R423: footprint Resistor_SMD:R_0402_1005Metric -> Resistor_SMD:R_0603_1608Metric
- R410: value 1M -> 100k
- R417, R418: value 4.7k -> 10k
Connections:
- net CODEC_VINR is gone; now on net CODEC_VIN: IC401.26 (VINR)
- net IN_BUF_IN_R is gone; now on an unnamed net: R410.1
- net GND: now also R410.2, J202.1 (Pin_1), J202.2 (Pin_2)
- net VCOM: no longer R410.2
- net OUT_BUF_OUT: now reaches R421.1, U406.1, U406.4 (-)
- net AUDIO_VINL renamed AUDIO_VIN
- net AUDIO_VIN: now also J202.2 (Pin_2)
- net AUDIO_VOUTL renamed AUDIO_VOUT
- net AUDIO_VOUT: now also J202.1 (Pin_1)
- net CODEC_VINL renamed CODEC_VIN
- net CODEC_VOUTL renamed CODEC_VOUT
- net CODEC_VOUTR: no longer names the net of IC401.18 (VOUTR+)
- net IN_AA_BUFF_IN_L renamed IN_AA_BUFF_IN
- net IN_AA_BUFF_OUT_L renamed IN_AA_BUFF_OUT
- net IN_BUF_IN_L renamed IN_BUF_IN
- net IN_BUF_OUT_L renamed IN_BUF_OUT
- net IN_RF_L renamed IN_RF
- net OUT_AA_BUFF_IN_L renamed OUT_AA_BUFF_IN
- net OUT_AA_BUFF_OUT_L renamed OUT_AA_BUFF_OUT
Other:
- note added: "3rd order Butterworth reconstruction filter. fc = 20kHz"
- note added: "Also use Channel Muting to further mute this pin"
- note added: "Termination Resistor"
- moved on the sheet: C402, C405, C419, C420, C421, C422, C423, C424, C428, C429, C430, C431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
