File: Power.kicad_sch (KiCad schematic)
At the start: 20 parts, among them J202 Screw_Terminal_01x02, U3 NCP718xSN500, U4 NCP1117-3.3_SOT223

Commit message: Refactoring
Parts:
- C201, C202, C203, C204: JLCPCB Part # (none) -> C108659
- C205, C206, C207, C208: JLCPCB Part # (none) -> C77081
- C209, C210: JLCPCB Part # (none) -> C90543
- D201, D202: JLCPCB Part # (none) -> C77336; JLCPCB Part# C77336 -> (none)
- D203: JLCPCB Part # (none) -> C908769; JLCPCB Part# C908769 -> (none)
- D204: JLCPCB Part # (none) -> C5123548
- FB302: JLCPCB Part # (none) -> C12391
- J202: JLCPCB Part # (none) -> C3029316; JLCPCB Part# C3029316 -> (none)
- R201: JLCPCB Part # (none) -> C17415
- R202: JLCPCB Part # (none) -> C102758
- U3: JLCPCB Part # (none) -> C892796; JLCPCB Part# C892796 -> (none)
- U4: JLCPCB Part # (none) -> C26537; JLCPCB Part# C26537 -> (none)
Changed lines of the file:
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@@
       (effects (font (size 1.27 1.27)) hide)
     )
-    (property "JLCPCB Part#" "" (at 169.545 69.215 0)
+    (property "JLCPCB Part #" "C108659" (at 169.545 69.215 0)
       (effects (font (size 1.27 1.27)) hide)
     )
@@
       (effects (font (size 1.27 1.27)) hide)
     )
-    (property "JLCPCB Part#" "" (at 191.135 69.215 0)
+    (property "JLCPCB Part #" "C108659" (at 191.135 69.215 0)
       (effects (font (size 1.27 1.27)) hide)
     )
@@
       (effects (font (size 1.27 1.27)) hide)
     )
-    (property "JLCPCB Part#" "" (at 201.93 69.215 0)
+    (property "JLCPCB Part #" "C108659" (at 201.93 69.215 0)
       (effects (font (size 1.27 1.27)) hide)
     )
@@
       (effects (font (size 1.27 1.27)) hide)
     )
-    (property "JLCPCB Part#" "C26537" (at 133.35 102.87 0)
+    (property "JLCPCB Part #" "C26537" (at 133.35 102.87 0)
       (effects (font (size 1.27 1.27)) hide)
     )
@@
       (effects (font (size 1.27 1.27)) hide)
     )
-    (property "JLCPCB Part#" "C77336" (at 112.395 55.88 0)
+    (property "JLCPCB Part #" "C77336" (at 112.395 55.88 0)
       (effects (font (size 1.27 1.27)) hide)
     )
@@
       (effects (font (size 1.27 1.27)) hide)
     )
-    (property "JLCPCB Part#" "" (at 117.475 69.85 0)
+    (property "JLCPCB Part #" "C77081" (at 117.475 69.85 0)
       (effects (font (size 1.27 1.27)) hide)
     )
@@
       (effects (font (size 1.27 1.27)) hide)
     )
-    (property "JLCPCB Part#" "" (at 162.56 102.87 0)
+    (property "JLCPCB Part #" "C102758" (at 162.56 102.87 0)
       (effects (font (size 1.27 1.27)) hide)
     )
@@
       (effects (font (size 1.27 1.27)) hide)
     )
-    (property "JLCPCB Part#" "C908769" (at 67.945 70.485 0)
+    (property "JLCPCB Part #" "C908769" (at 67.945 70.485 0)
       (effects (font (size 1.27 1.27)) hide)
     )
@@
       (effects (font (size 1.27 1.27)) hide)
     )
-    (property "JLCPCB Part#" "" (at 162.56 62.865 0)
+    (property "JLCPCB Part #" "C17415" (at 162.56 62.865 0)
       (effects (font (size 1.27 1.27)) hide)
     )
@@
       (effects (font (size 1.27 1.27)) hide)
     )
-    (property "JLCPCB Part#" "" (at 146.685 109.22 0)
+    (property "JLCPCB Part #" "C90543" (at 146.685 109.22 0)
       (effects (font (size 1.27 1.27)) hide)
     )
@@
       (effects (font (size 1.27 1.27)) hide)
     )
-    (property "JLCPCB Part#" "C892796" (at 133.35 65.405 0)
+    (property "JLCPCB Part #" "C892796" (at 133.35 65.405 0)
       (effects (font (size 1.27 1.27)) hide)
     )
@@
       (effects (font (size 1.27 1.27)) hide)
     )
-    (property "JLCPCB Part#" "" (at 118.11 109.855 0)
+    (property "JLCPCB Part #" "C90543" (at 118.11 109.855 0)
       (effects (font (size 1.27 1.27)) hide)
     )
@@
       (effects (font (size 1.27 1.27)) hide)
     )
-    (property "JLCPCB Part#" "" (at 94.615 62.865 0)
+    (property "JLCPCB Part #" "C12391" (at 94.615 62.865 0)
       (effects (font (size 1.27 1.27)) hide)
     )
@@
       (effects (font (size 1.27 1.27)) hide)
     )
-    (property "JLCPCB Part#" "C3029316" (at 49.53 65.405 0)
+    (property "JLCPCB Part #" "C3029316" (at 49.53 65.405 0)
       (effects (font (size 1.27 1.27)) hide)
     )
@@
       (effects (font (size 1.27 1.27)) hide)
     )
-    (property "JLCPCB Part#" "" (at 147.32 69.85 0)
+    (property "JLCPCB Part #" "C77081" (at 147.32 69.85 0)
       (effects (font (size 1.27 1.27)) hide)
     )
@@
       (effects (font (size 1.27 1.27)) hide)
     )
-    (property "JLCPCB Part#" "" (at 102.235 69.85 0)
+    (property "JLCPCB Part #" "C77081" (at 102.235 69.85 0)
       (effects (font (size 1.27 1.27)) hide)
     )
@@
       (effects (font (size 1.27 1.27)) hide)
     )
-    (property "JLCPCB Part#" "" (at 172.085 109.22 0)
+    (property "JLCPCB Part #" "C5123548" (at 172.085 109.22 0)
       (effects (font (size 1.27 1.27)) hide)
     )
@@
       (effects (font (size 1.27 1.27)) hide)
     )
-    (property "JLCPCB Part#" "" (at 180.34 69.215 0)
+    (property "JLCPCB Part #" "C108659" (at 180.34 69.215 0)
       (effects (font (size 1.27 1.27)) hide)
     )
@@
       (effects (font (size 1.27 1.27)) hide)
     )
-    (property "JLCPCB Part#" "" (at 87.63 69.85 0)
+    (property "JLCPCB Part #" "C77081" (at 87.63 69.85 0)
       (effects (font (size 1.27 1.27)) hide)
     )
@@
       (effects (font (size 1.27 1.27)) hide)
     )
-    (property "JLCPCB Part#" "C77336" (at 78.105 62.865 0)
-      (effects (font (size 1.27 1.27)) hide)
-    )
+    (property "JLCPCB Part #" "C77336" (at 78.105 62.865 0)
+      (effects (font (size 1.27 1.27)) hide)
+    )
